Commit message: Converted environment to MuJoCo

File: quadrupedX.urdf (robot description, URDF)
Before this commit: robot ROS2, 17 links, 16 joints
Links:
- link Back_Left_Foot_1: geometry collision mesh filename=meshes/Back_Left_Foot_1.stl scale=0.001 0.001 0.001; visual mesh filename=meshes/Back_Left_Foot_1.stl scale=0.001 0.001 0.001
- link Back_Left_Lower_1: geometry collision mesh filename=meshes/Back_Left_Lower_1.stl scale=0.001 0.001 0.001; visual mesh filename=meshes/Back_Left_Lower_1.stl scale=0.001 0.001 0.001
- link Back_Left_Shoulder_1: geometry collision mesh filename=meshes/Back_Left_Shoulder_1.stl scale=0.001 0.001 0.001; visual mesh filename=meshes/Back_Left_Shoulder_1.stl scale=0.001 0.001 0.001
- link Back_Left_Upper_1: geometry collision mesh filename=meshes/Back_Left_Upper_1.stl scale=0.001 0.001 0.001; visual mesh filename=meshes/Back_Left_Upper_1.stl scale=0.001 0.001 0.001
- link Back_Right_Foot_1: geometry collision mesh filename=meshes/Back_Right_Foot_1.stl scale=0.001 0.001 0.001; visual mesh filename=meshes/Back_Right_Foot_1.stl scale=0.001 0.001 0.001
- link Back_Right_Lower_1: geometry collision mesh filename=meshes/Back_Right_Lower_1.stl scale=0.001 0.001 0.001; visual mesh filename=meshes/Back_Right_Lower_1.stl scale=0.001 0.001 0.001
- link Back_Right_Shoulder_1: geometry collision mesh filename=meshes/Back_Right_Shoulder_1.stl scale=0.001 0.001 0.001; visual mesh filename=meshes/Back_Right_Shoulder_1.stl scale=0.001 0.001 0.001
- link Back_Right_Upper_1: geometry collision mesh filename=meshes/Back_Right_Upper_1.stl scale=0.001 0.001 0.001; visual mesh filename=meshes/Back_Right_Upper_1.stl scale=0.001 0.001 0.001
- link Fright_Right_Shoulder_1: geometry collision mesh filename=meshes/Fright_Right_Shoulder_1.stl scale=0.001 0.001 0.001; visual mesh filename=meshes/Fright_Right_Shoulder_1.stl scale=0.001 0.001 0.001
- link Front_Left_Foot_1: geometry collision mesh filename=meshes/Front_Left_Foot_1.stl scale=0.001 0.001 0.001; visual mesh filename=meshes/Front_Left_Foot_1.stl scale=0.001 0.001 0.001
- link Front_Left_Lower_1: geometry collision mesh filename=meshes/Front_Left_Lower_1.stl scale=0.001 0.001 0.001; visual mesh filename=meshes/Front_Left_Lower_1.stl scale=0.001 0.001 0.001
- link Front_Left_Shoulder_1: geometry collision mesh filename=meshes/Front_Left_Shoulder_1.stl scale=0.001 0.001 0.001; visual mesh filename=meshes/Front_Left_Shoulder_1.stl scale=0.001 0.001 0.001
- link Front_Left_Upper_1: geometry collision mesh filename=meshes/Front_Left_Upper_1.stl scale=0.001 0.001 0.001; visual mesh filename=meshes/Front_Left_Upper_1.stl scale=0.001 0.001 0.001
- link Front_Right_Foot_1: geometry collision mesh filename=meshes/Front_Right_Foot_1.stl scale=0.001 0.001 0.001; visual mesh filename=meshes/Front_Right_Foot_1.stl scale=0.001 0.001 0.001
- link Front_Right_Lower_1: geometry collision mesh filename=meshes/Front_Right_Lower_1.stl scale=0.001 0.001 0.001; visual mesh filename=meshes/Front_Right_Lower_1.stl scale=0.001 0.001 0.001
- link Front_Right_Upper_1: geometry collision mesh filename=meshes/Front_Right_Upper_1.stl scale=0.001 0.001 0.001; visual mesh filename=meshes/Front_Right_Upper_1.stl scale=0.001 0.001 0.001
- link base_link: geometry collision mesh filename=meshes/base_link.stl scale=0.001 0.001 0.001; visual mesh filename=meshes/base_link.stl scale=0.001 0.001 0.001
